File: Hardware/Schematic/Arduino_Buck.sch (KiCad schematic (older format))
At the start: 9 parts

Commit message: Added Power Board Rev. B
Parts:
- C17: renamed from C?; value 2.2uF -> 2U2; footprint Resistor_SMD:R_0805_2012Metric_Pad1.15x1.40mm_HandSolder -> Capacitor_SMD:C_0805_2012Metric_Pad1.15x1.40mm_HandSolder; Manufacturer_Part_Number (none) -> C0805X5R225K500NT
- D3: renamed from D?; value SS34 -> SS24; footprint Diode_SMD:D_SMC_Handsoldering -> ArduinoLamp:D_SMA_Handsoldering_Shortened; Mouser Part Number (none) -> C181203
- L4: renamed from L?; value L -> 330U; footprint (none) -> ArduinoLamp:SLD10; Manufacturer_Part_Number (none) -> SLD10D40S331MTT
- Q3: renamed from Q?; Manufacturer_Part_Number (none) -> 2N7000
- Q4: renamed from Q?; value TSM2301ACX -> PJM2301PSA-S; Manufacturer_Part_Number (none) -> PJM2301PSA-S
- R16, R17: renamed from R?; value 105k -> 105K; Manufacturer_Part_Number (none) -> RC0603FR-07105KL
- R18: renamed from R?; value 25.5k -> 25K5; Manufacturer_Part_Number (none) -> RS-05K2552FT
- R19: renamed from R?; value 1.15k -> 1K15; Manufacturer_Part_Number (none) -> RS-03K1151FT
Changed lines of the file:
@@
 $Descr A4 11693 8268
 encoding utf-8
-Sheet 6 7
+Sheet 5 7
 Title ""
 Date ""
@@
 PWM
 $Comp
-L Transistor_FET:TSM2301ACX Q?
+L Transistor_FET:TSM2301ACX Q4
 U 1 1 5F8E71B4
 P 5500 3700
-F 0 "Q?" H 5704 3746 50  0000 L CNN
-F 1 "TSM2301ACX" H 5704 3655 50  0000 L CNN
+F 0 "Q4" H 5704 3746 50  0000 L CNN
+F 1 "PJM2301PSA-S" H 5704 3655 50  0000 L CNN
 F 2 "Package_TO_SOT_SMD:SOT-23" H 5700 3625 50  0001 L CIN
 F 3 "https://www.taiwansemi.com/products/datasheet/TSM2301A_C15.pdf" H 5500 3700 50  0001 L CNN
+F 4 "PJM2301PSA-S" H 5500 3700 50  0001 C CNN "Manufacturer_Part_Number"
 	1    5500 3700
 	0    -1   -1   0
 $EndComp
 $Comp
-L Device:L L?
+L Device:L L4
 U 1 1 5F8E9295
 P 6250 3600
-F 0 "L?" V 6440 3600 50  0000 C CNN
-F 1 "L" V 6349 3600 50  0000 C CNN
-F 2 "" H 6250 3600 50  0001 C CNN
+F 0 "L4" V 6440 3600 50  0000 C CNN
+F 1 "330U" V 6349 3600 50  0000 C CNN
+F 2 "ArduinoLamp:SLD10" H 6250 3600 50  0001 C CNN
 F 3 "~" H 6250 3600 50  0001 C CNN
+F 4 "SLD10D40S331MTT" H 6250 3600 50  0001 C CNN "Manufacturer_Part_Number"
 	1    6250 3600
 	0    -1   -1   0
 $EndComp
 $Comp
-L Device:D_Schottky D?
+L Device:D_Schottky D3
 U 1 1 5F8E9922
 P 5950 4000
-F 0 "D?" V 5904 4080 50  0000 L CNN
-F 1 "SS34" V 5995 4080 50  0000 L CNN
-F 2 "Diode_SMD:D_SMC_Handsoldering" H 5950 4000 50  0001 C CNN
+F 0 "D3" V 5904 4080 50  0000 L CNN
+F 1 "SS24" V 5995 4080 50  0000 L CNN
+F 2 "ArduinoLamp:D_SMA_Handsoldering_Shortened" H 5950 4000 50  0001 C CNN
 F 3 "~" H 5950 4000 50  0001 C CNN
+F 4 "C181203" H 5950 4000 50  0001 C CNN "Mouser Part Number"
 	1    5950 4000
 	0    1    1    0
 $EndComp
 $Comp
-L Device:C C?
+L Device:C C17
 U 1 1 5F8EC349
 P 6550 4000
-F 0 "C?" H 6665 4046 50  0000 L CNN
-F 1 "2.2uF" H 6665 3955 50  0000 L CNN
-F 2 "Resistor_SMD:R_0805_2012Metric_Pad1.15x1.40mm_HandSolder" H 6588 3850 50  0001 C CNN
+F 0 "C17" H 6665 4046 50  0000 L CNN
+F 1 "2U2" H 6665 3955 50  0000 L CNN
+F 2 "Capacitor_SMD:C_0805_2012Metric_Pad1.15x1.40mm_HandSolder" H 6588 3850 50  0001 C CNN
 F 3 "~" H 6550 4000 50  0001 C CNN
+F 4 "C0805X5R225K500NT" H 6550 4000 50  0001 C CNN "Manufacturer_Part_Number"
 	1    6550 4000
 	1    0    0    -1
 $EndComp
 $Comp
-L Device:R R?
+L Device:R R18
 U 1 1 5F8ECD7F
 P 6950 3850
-F 0 "R?" H 7020 3896 50  0000 L CNN
-F 1 "25.5k" H 7020 3805 50  0000 L CNN
+F 0 "R18" H 7020 3896 50  0000 L CNN
+F 1 "25K5" H 7020 3805 50  0000 L CNN
 F 2 "Resistor_SMD:R_0603_1608Metric_Pad1.05x0.95mm_HandSolder" V 6880 3850 50  0001 C CNN
 F 3 "~" H 6950 3850 50  0001 C CNN
+F 4 "RS-05K2552FT" H 6950 3850 50  0001 C CNN "Manufacturer_Part_Number"
 	1    6950 3850
 	1    0    0    -1
 $EndComp
 $Comp
-L Device:R R?
+L Device:R R19
 U 1 1 5F8ED5C2
 P 6950 4200
-F 0 "R?" H 7020 4246 50  0000 L CNN
-F 1 "1.15k" H 7020 4155 50  0000 L CNN
+F 0 "R19" H 7020 4246 50  0000 L CNN
+F 1 "1K15" H 7020 4155 50  0000 L CNN
 F 2 "Resistor_SMD:R_0603_1608Metric_Pad1.05x0.95mm_HandSolder" V 6880 4200 50  0001 C CNN
 F 3 "~" H 6950 4200 50  0001 C CNN
+F 4 "RS-03K1151FT" H 6950 4200 50  0001 C CNN "Manufacturer_Part_Number"
 	1    6950 4200
 	1    0    0    -1
@@
 	6950 4050 6950 4000
 $Comp
-L Transistor_FET:2N7000 Q?
+L Transistor_FET:2N7000 Q3
 U 1 1 5F8F3832
 P 5400 4100
-F 0 "Q?" H 5604 4146 50  0000 L CNN
+F 0 "Q3" H 5604 4146 50  0000 L CNN
 F 1 "2N7000" H 5604 4055 50  0000 L CNN
 F 2 "Package_TO_SOT_THT:TO-92_Inline" H 5600 4025 50  0001 L CIN
 F 3 "https://www.fairchildsemi.com/datasheets/2N/2N7000.pdf" H 5400 4100 50  0001 L CNN
+F 4 "2N7000" H 5400 4100 50  0001 C CNN "Manufacturer_Part_Number"
 	1    5400 4100
 	1    0    0    -1
@@
 	4700 4100 5050 4100
 $Comp
-L Device:R R?
+L Device:R R17
 U 1 1 5F8F67F8
 P 5050 4250
-F 0 "R?" H 5120 4296 50  0000 L CNN
-F 1 "105k" H 5120 4205 50  0000 L CNN
+F 0 "R17" H 5120 4296 50  0000 L CNN
+F 1 "105K" H 5120 4205 50  0000 L CNN
 F 2 "Resistor_SMD:R_0603_1608Metric_Pad1.05x0.95mm_HandSolder" V 4980 4250 50  0001 C CNN
 F 3 "~" H 5050 4250 50  0001 C CNN
+F 4 "RC0603FR-07105KL" H 5050 4250 50  0001 C CNN "Manufacturer_Part_Number"
 	1    5050 4250
 	1    0    0    -1
@@
 	4700 3900 4900 3900
 $Comp
-L Device:R R?
+L Device:R R16
 U 1 1 5F8FA0B3
 P 5050 3750
-F 0 "R?" H 5120 3796 50  0000 L CNN
-F 1 "105k" H 5120 3705 50  0000 L CNN
+F 0 "R16" H 5120 3796 50  0000 L CNN
+F 1 "105K" H 5120 3705 50  0000 L CNN
 F 2 "Resistor_SMD:R_0603_1608Metric_Pad1.05x0.95mm_HandSolder" V 4980 3750 50  0001 C CNN
 F 3 "~" H 5050 3750 50  0001 C CNN
+F 4 "RC0603FR-07105KL" H 5050 3750 50  0001 C CNN "Manufacturer_Part_Number"
 	1    5050 3750
 	1    0    0    -1
