File: Hardware/Schematic/LM3481.sch (KiCad schematic (older format))
At the start: 21 parts, among them IC1 LM3481MM, Q1 2N7000, Q2 AO4264E

Commit message: Added Power Board Rev. B
Parts:
- added R9: 20, Resistor_SMD:R_0603_1608Metric_Pad1.05x0.95mm_HandSolder, symbol Device:R
- C2: value 2.2uF -> 2U2; Manufacturer_Part_Number (none) -> C0805X5R225K500NT
- C3: value 1.2nF -> 1N2; Manufacturer_Part_Number (none) -> C1608C0G1H122JT000N
- C4: value 330nF -> 330N; Manufacturer_Part_Number (none) -> TCC0603X7R334K500CT
- C5: value 470nF -> 470N; Manufacturer_Part_Number (none) -> 0603B474K100CT
- C6: value 4.7uF -> 4U7; footprint Capacitor_SMD:C_0603_1608Metric_Pad1.05x0.95mm_HandSolder -> Capacitor_SMD:C_1206_3216Metric_Pad1.42x1.75mm_HandSolder; Manufacturer_Part_Number (none) -> GRM31CR71H475KA12L
- C7: value 100nF -> 100N; Manufacturer_Part_Number (none) -> CL10B104KB8NNNC
- C8: value 470pF -> 470P; Manufacturer_Part_Number (none) -> TCC0603COG471J500CT
- C9: value 2.2u -> 2U2; Manufacturer_Part_Number (none) -> C0805X5R225K500NT
- D1: value D_Schottky -> SS510; footprint Diode_SMD:D_SMC_Handsoldering -> ArduinoLamp:D_SMC_Handsoldering_Shortened; Mouser Part Number (none) -> C19229
- IC1: footprint LED Power Board parts:SOP50P490X110-10N -> Package_SO:VSSOP-10_3x3mm_P0.5mm
- L1: value SRF1260-6R8YCT-ND -> SRF1260-6R8; footprint Inductor_SMD:L_Bourns_SRF1260 -> ArduinoLamp:L_Bourns_SRF1260_HandSoldering; symbol Device:L_Coupled -> ArduinoLamp:L_Coupled_1324; Manufacturer_Part_Number (none) -> SRF1260-6R8
- Q1: Manufacturer_Part_Number (none) -> 2N7000
- Q2: footprint Package_SO:SOIC-8_3.9x4.9mm_P1.27mm -> Package_SO:SO-8_3.9x4.9mm_P1.27mm; Manufacturer_Part_Number (none) -> AO4264E
- R1, R7: value 105k -> 105K; Manufacturer_Part_Number (none) -> RC0603FR-07105KL
- R2, R4: value 25.5k -> 25K5; footprint Resistor_SMD:R_0805_2012Metric_Pad1.15x1.40mm_HandSolder -> Resistor_SMD:R_0603_1608Metric_Pad1.05x0.95mm_HandSolder; Manufacturer_Part_Number (none) -> RS-05K2552FT
- R3: Manufacturer_Part_Number (none) -> 0603WAF4420T5E
- R5: Manufacturer_Part_Number (none) -> 0603WAJ0101T5E
- R6: value 0.006 -> 0R006; Manufacturer_Part_Number (none) -> PA1206FRF070R006L
- R8: value 6.49k -> 6K49; Manufacturer_Part_Number (none) -> RS-03K6491FT
Connections:
- net labels added: GNDA, LM3481_VIN
- wire segments 85 -> 93
Other:
- moved on the sheet: R4, R6
