File: Hardware/Schematic/Power Board V2.sch (KiCad schematic (older format))
At the start: 7 parts

Commit message: Added Power Board Rev. B
Parts:
- removed J?: POWER_IN, symbol Connector_Generic:Conn_01x02
- removed R?: 105k, Resistor_SMD:R_0603_1608Metric_Pad1.05x0.95mm_HandSolder, symbol Device:R
- added C10, C11, C24: 100N, Capacitor_SMD:C_0603_1608Metric_Pad1.05x0.95mm_HandSolder, symbol Device:C
- added C23: CP, Capacitor_THT:CP_Radial_D10.0mm_P5.00mm, symbol Device:CP
- added C25, C26: CP, Capacitor_THT:CP_Radial_D6.3mm_P2.50mm, symbol Device:CP
- added H1, H2, H3, H4: MountingHole_Pad, MountingHole:MountingHole_3.2mm_M3_Pad_Via, symbol Mechanical:MountingHole_Pad
- added J1, J2, J3, J4: Conn_01x02, Connector_JST:JST_XH_B2B-XH-A_1x02_P2.50mm_Vertical, symbol Connector_Generic:Conn_01x02
- added J5: Conn_02x05_Top_Bottom, Connector_IDC:IDC-Header_2x05_P2.54mm_Vertical, symbol Connector_Generic:Conn_02x05_Top_Bottom
- added R22, R24, R28: 25K5, Resistor_SMD:R_0603_1608Metric_Pad1.05x0.95mm_HandSolder, symbol Device:R
- added R23, R25: 1K15, Resistor_SMD:R_0603_1608Metric_Pad1.05x0.95mm_HandSolder, symbol Device:R
- added TP1: GND, TestPoint:TestPoint_Pad_D1.5mm, symbol Connector:TestPoint
- added TP2: +22V, TestPoint:TestPoint_Pad_D1.5mm, symbol Connector:TestPoint
- added TP3: +5V, TestPoint:TestPoint_Pad_D1.5mm, symbol Connector:TestPoint
- added TP4: B_CTRL, TestPoint:TestPoint_Pad_D1.5mm, symbol Connector:TestPoint
- added TP5: Y_CTRL, TestPoint:TestPoint_Pad_D1.5mm, symbol Connector:TestPoint
- C1: renamed from C?; value 330uF 50V -> 220U; footprint (none) -> Capacitor_THT:CP_Radial_D8.0mm_P3.50mm
- R10: renamed from R?; value 8.45k -> 8K45; Manufacturer_Part_Number (none) -> RS-03K8451FT
- R11, R13: renamed from R?; value 1.58k -> 1K15; Manufacturer_Part_Number (none) -> RS-03K1151FT
- R12: renamed from R?; value 25.5k -> 25K5; Manufacturer_Part_Number (none) -> RS-05K2552FT
Connections:
- net +5V: now also C25.1, J5.1 (Pin_1), R28.1, TP3.1
- net FAN_FB: now also C24.1, J5.10 (Pin_10)
- net GNDPWR: now also C10.2, C11.2, C23.2, C24.2, C25.2, C26.2, H1.1, H2.1, H3.1, H4.1, J1.1 (Pin_1), J2.2 (Pin_2), J5.4 (Pin_4), J5.8 (Pin_8), R23.2, R25.2, TP1.1
- net PWM Fan Control/FAN: now also J2.1 (Pin_1)
- net PWR_EN: now also J5.5 (Pin_5), R28.2
- net VIN: now also J1.2 (Pin_2), R22.1
- net Fan Power Supply/VOUT renamed +13V9
- net +13V9: now also C26.1
- new net +22V: C23.1, R24.1, TP2.1
- new net BLUE_CTRL: J5.7 (Pin_7), TP4.1
- new net Cold White Driver/LED+: J4.1 (Pin_1)
- new net Cold White Driver/LED-: J4.2 (Pin_2)
- new net FAN_CTRL: J5.9 (Pin_9)
- new net VIN_FB: C10.1, J5.2 (Pin_2), R22.2, R23.1
- new net VOUT_FB: C11.1, J5.3 (Pin_3), R24.2, R25.1
- new net Warm White Driver/LED+: J3.1 (Pin_1)
- new net Warm White Driver/LED-: J3.2 (Pin_2)
- new net YELLOW_CTRL: J5.6 (Pin_6), TP5.1
Other:
- moved on the sheet: R10, R11, R12, R13
